File: hardware/pcb/copyMe84.kicad_pcb (KiCad board)
At the start: 2 copper layers, 83.8 x 57.1 mm, 16 parts, among them IC1 ATTINY84A-P

Commit message: V2
Parts:
- removed S1: RED, Switch - TS0B22:Tactile Switch - TS0B22
- removed S2: BLUE, Switch - TS0B22:Tactile Switch - TS0B22
- removed S3: YELLOW, Switch - TS0B22:Tactile Switch - TS0B22
- removed S4: GREEN, Switch - TS0B22:Tactile Switch - TS0B22
- added SW1: KFC-012-7.3, tfhSwitches:KFC-012-7.3, F.Cu at (111.8, 125.7)
- added SW2: KFC-012-7.3, tfhSwitches:KFC-012-7.3, F.Cu at (132.1, 125.7)
- added SW3: KFC-012-7.3, tfhSwitches:KFC-012-7.3, F.Cu at (152.4, 125.7)
- added SW4: KFC-012-7.3, tfhSwitches:KFC-012-7.3, F.Cu at (172.7, 125.7)
- BT1: value Battery -> CR2477; footprint BatteryHolder2462:Battery Holder - Keystone 2462 -> TFH Batteries:CR2477
- R1, R2, R3, R4, R5: value 500 -> 220
- moved BT1 10.9 mm to (125.7, 90.2), turned to 90 degrees
Routing:
- net Earth: track 226.0 -> 242.2 mm, vias 2 -> 0
- net /ledRED: track 14.8 -> 22.7 mm
- net /swYELLOW: track 127.3 -> 119.8 mm
- net /swRED: track 69.9 -> 74.5 mm
- net /swGREEN: track 90.3 -> 88.0 mm
- net Net-(BT1-Pad1): track 12.0 -> 10.1 mm
- net /swBLUE: track 103.2 -> 104.4 mm
- net (no net): track 0.11 -> 0.00 mm, vias 0 -> 1
Other:
- board text added: "Ver. 2"
- board text removed: "Ver. 1"

Commit message: V2.1
Connections:
- IC1 pad 4: /ledYELLOW -> Net-(IC1-Pad4)
- IC1 pad 5: /ledGREEN -> /ledYELLOW
- IC1 pad 6: Net-(IC1-Pad6) -> /ledGREEN
Routing:
- net /ledYELLOW: track 21.9 -> 18.6 mm
- net /ledGREEN: track 38.7 -> 37.7 mm
Other:
- board text added: "Ver. 2.1"
- board text removed: "Ver. 2"
