File: hardware/pcb/copyMe84.sch (KiCad schematic (older format))
At the start: 16 parts, among them IC1 ATTINY84A-P

Commit message: updates
Parts:
- BT1: value Battery -> CR2477
- R1, R2, R3, R4, R5: value 500 -> 220
Changed lines of the file:
@@
 P 7000 3400
 F 0 "R1" V 7080 3400 50  0000 C CNN
-F 1 "500" V 7000 3400 50  0000 C CNN
+F 1 "220" V 7000 3400 50  0000 C CNN
 F 2 "Resistors_ThroughHole:Resistor_Horizontal_RM10mm" V 6930 3400 50  0001 C CNN
 F 3 "" H 7000 3400 50  0000 C CNN
@@
 P 7350 3400
 F 0 "R2" V 7430 3400 50  0000 C CNN
-F 1 "500" V 7350 3400 50  0000 C CNN
+F 1 "220" V 7350 3400 50  0000 C CNN
 F 2 "Resistors_ThroughHole:Resistor_Horizontal_RM10mm" V 7280 3400 50  0001 C CNN
 F 3 "" H 7350 3400 50  0000 C CNN
@@
 P 7700 3400
 F 0 "R3" V 7780 3400 50  0000 C CNN
-F 1 "500" V 7700 3400 50  0000 C CNN
+F 1 "220" V 7700 3400 50  0000 C CNN
 F 2 "Resistors_ThroughHole:Resistor_Horizontal_RM10mm" V 7630 3400 50  0001 C CNN
 F 3 "" H 7700 3400 50  0000 C CNN
@@
 P 8050 3400
 F 0 "R4" V 8130 3400 50  0000 C CNN
-F 1 "500" V 8050 3400 50  0000 C CNN
+F 1 "220" V 8050 3400 50  0000 C CNN
 F 2 "Resistors_ThroughHole:Resistor_Horizontal_RM10mm" V 7980 3400 50  0001 C CNN
 F 3 "" H 8050 3400 50  0000 C CNN
@@
 P 8750 3400
 F 0 "R5" V 8830 3400 50  0000 C CNN
-F 1 "500" V 8750 3400 50  0000 C CNN
+F 1 "220" V 8750 3400 50  0000 C CNN
 F 2 "Resistors_ThroughHole:Resistor_Horizontal_RM10mm" V 8680 3400 50  0001 C CNN
 F 3 "" H 8750 3400 50  0000 C CNN
@@
 P 2150 3900
 F 0 "BT1" H 2250 3950 50  0000 L CNN
-F 1 "Battery" H 2250 3850 50  0000 L CNN
+F 1 "CR2477" H 2250 3850 50  0000 L CNN
 F 2 "BatteryHolder2462:Battery Holder - Keystone 2462" V 2150 3940 50  0001 C CNN
 F 3 "" V 2150 3940 50  0000 C CNN

Commit message: V2
Parts:
- removed S1: RED, Switch - TS0B22:Tactile Switch - TS0B22, symbol Switch_Tactile_-_TS0B22
- removed S2: BLUE, Switch - TS0B22:Tactile Switch - TS0B22, symbol Switch_Tactile_-_TS0B22
- removed S3: YELLOW, Switch - TS0B22:Tactile Switch - TS0B22, symbol Switch_Tactile_-_TS0B22
- removed S4: GREEN, Switch - TS0B22:Tactile Switch - TS0B22, symbol Switch_Tactile_-_TS0B22
- added SW1, SW2, SW3, SW4: KFC-012-7.3, tfhSwitches:KFC-012-7.3, symbol KFC-012-7.3
- BT1: footprint BatteryHolder2462:Battery Holder - Keystone 2462 -> TFH Batteries:CR2477
Connections:
- wire segments 37 -> 45
- no-connect marks 11 -> 8
Changed lines of the file:
@@
 LIBS:IHE
 LIBS:switch_tactile_-_ts0b22
+LIBS:tfhSwitches
 LIBS:copyMe84-cache
 EELAYER 25 0
@@
 F 0 "BT1" H 2250 3950 50  0000 L CNN
 F 1 "CR2477" H 2250 3850 50  0000 L CNN
-F 2 "BatteryHolder2462:Battery Holder - Keystone 2462" V 2150 3940 50  0001 C CNN
+F 2 "TFH Batteries:CR2477" V 2150 3940 50  0001 C CNN
 F 3 "" V 2150 3940 50  0000 C CNN
 	1    2150 3900
@@
 	8050 4050 8050 4150
 $Comp
-L Switch_Tactile_-_TS0B22 S1
-U 1 1 5732B6FA
-P 6900 5150
-F 0 "S1" H 7050 5000 60  0000 C CNN
-F 1 "RED" H 6900 5350 60  0000 C CNN
-F 2 "Switch - TS0B22:Tactile Switch - TS0B22" H 6900 5150 60  0001 C CNN
-F 3 "" H 6900 5150 60  0000 C CNN
-	1    6900 5150
-	0    -1   -1   0
-$EndComp
-$Comp
-L Switch_Tactile_-_TS0B22 S2
-U 1 1 5732B826
-P 7800 5200
-F 0 "S2" H 7950 5050 60  0000 C CNN
-F 1 "BLUE" H 7800 5400 60  0000 C CNN
-F 2 "Switch - TS0B22:Tactile Switch - TS0B22" H 7800 5200 60  0001 C CNN
-F 3 "" H 7800 5200 60  0000 C CNN
-	1    7800 5200
-	0    -1   -1   0
-$EndComp
-$Comp
-L Switch_Tactile_-_TS0B22 S3
-U 1 1 5732B86A
-P 8600 5150
-F 0 "S3" H 8750 5000 60  0000 C CNN
-F 1 "YELLOW" H 8600 5350 60  0000 C CNN
-F 2 "Switch - TS0B22:Tactile Switch - TS0B22" H 8600 5150 60  0001 C CNN
-F 3 "" H 8600 5150 60  0000 C CNN
-	1    8600 5150
-	0    -1   -1   0
-$EndComp
-$Comp
-L Switch_Tactile_-_TS0B22 S4
-U 1 1 5732B8B7
-P 9600 5150
-F 0 "S4" H 9750 5000 60  0000 C CNN
-F 1 "GREEN" H 9600 5350 60  0000 C CNN
-F 2 "Switch - TS0B22:Tactile Switch - TS0B22" H 9600 5150 60  0001 C CNN
-F 3 "" H 9600 5150 60  0000 C CNN
-	1    9600 5150
-	0    -1   -1   0
-$EndComp
-$Comp
 L Earth #PWR09
 U 1 1 5732BC63
-P 6950 5950
-F 0 "#PWR09" H 6950 5700 50  0001 C CNN
-F 1 "Earth" H 6950 5800 50  0001 C CNN
-F 2 "" H 6950 5950 50  0000 C CNN
-F 3 "" H 6950 5950 50  0000 C CNN
-	1    6950 5950
+P 6250 5850
+F 0 "#PWR09" H 6250 5600 50  0001 C CNN
+F 1 "Earth" H 6250 5700 50  0001 C CNN
+F 2 "" H 6250 5850 50  0000 C CNN
+F 3 "" H 6250 5850 50  0000 C CNN
+	1    6250 5850
 	1    0    0    -1
 $EndComp
@@
 L Earth #PWR010
 U 1 1 5732BC9E
-P 7850 5950
-F 0 "#PWR010" H 7850 5700 50  0001 C CNN
-F 1 "Earth" H 7850 5800 50  0001 C CNN
-F 2 "" H 7850 5950 50  0000 C CNN
-F 3 "" H 7850 5950 50  0000 C CNN
-	1    7850 5950
+P 7350 5850
+F 0 "#PWR010" H 7350 5600 50  0001 C CNN
+F 1 "Earth" H 7350 5700 50  0001 C CNN
+F 2 "" H 7350 5850 50  0000 C CNN
+F 3 "" H 7350 5850 50  0000 C CNN
+	1    7350 5850
 	1    0    0    -1
 $EndComp
@@
 L Earth #PWR011
 U 1 1 5732BCD9
-P 8650 5950
-F 0 "#PWR011" H 8650 5700 50  0001 C CNN
-F 1 "Earth" H 8650 5800 50  0001 C CNN
-F 2 "" H 8650 5950 50  0000 C CNN
-F 3 "" H 8650 5950 50  0000 C CNN
-	1    8650 5950
+P 8450 5850
+F 0 "#PWR011" H 8450 5600 50  0001 C CNN
+F 1 "Earth" H 8450 5700 50  0001 C CNN
+F 2 "" H 8450 5850 50  0000 C CNN
+F 3 "" H 8450 5850 50  0000 C CNN
+	1    8450 5850
 	1    0    0    -1
 $EndComp
@@
 L Earth #PWR012
 U 1 1 5732BD14
-P 9650 5950
-F 0 "#PWR012" H 9650 5700 50  0001 C CNN
-F 1 "Earth" H 9650 5800 50  0001 C CNN
-F 2 "" H 9650 5950 50  0000 C CNN
-F 3 "" H 9650 5950 50  0000 C CNN
-	1    9650 5950
-	1    0    0    -1
-$EndComp
-Wire Wire Line
-	6950 5400 6950 5950
-Wire Wire Line
-	7850 5450 7850 5950
-Wire Wire Line
-	9650 5400 9650 5950
-Wire Wire Line
-	6950 4550 6950 4900
-Wire Wire Line
-	7850 4550 7850 4950
-Wire Wire Line
-	8650 4550 8650 4900
-Wire Wire Line
-	9650 4550 9650 4900
-Text Label 6950 4850 1    60   ~ 0
+P 9550 5850
+F 0 "#PWR012" H 9550 5600 50  0001 C CNN
+F 1 "Earth" H 9550 5700 50  0001 C CNN
+F 2 "" H 9550 5850 50  0000 C CNN
+F 3 "" H 9550 5850 50  0000 C CNN
+	1    9550 5850
+	1    0    0    -1
+$EndComp
+Wire Wire Line
+	6250 4650 6250 5200
+Wire Wire Line
+	7350 4650 7350 5200
+Text Label 6250 5000 1    60   ~ 0
 swRED
-Text Label 7850 4850 1    60   ~ 0
+Text Label 7350 5050 1    60   ~ 0
 swBLUE
-Text Label 8650 4850 1    60   ~ 0
+Text Label 9350 5050 1    60   ~ 0
 swYELLOW
-NoConn ~ 6850 4900
-NoConn ~ 6850 5400
-Text Label 9650 4850 1    60   ~ 0
+Text Label 10450 5050 1    60   ~ 0
 swGREEN
-NoConn ~ 7750 4950
-NoConn ~ 7750 5450
-NoConn ~ 8550 4900
-NoConn ~ 8550 5400
-NoConn ~ 9550 4900
-NoConn ~ 9550 5400
-Wire Wire Line
-	8650 5400 8650 5950
 Text Label 5300 4450 0    60   ~ 0
 ledGREEN
@@
 Text Label 5300 3850 0    60   ~ 0
 swGREEN
+$Comp
+L KFC-012-7.3 SW1
+U 1 1 5780D7F1
+P 6700 5400
+F 0 "SW1" H 6700 5050 60  0000 C CNN
+F 1 "KFC-012-7.3" H 6700 5750 60  0000 C CNN
+F 2 "tfhSwitches:KFC-012-7.3" H 6700 5400 60  0001 C CNN
+F 3 "" H 6700 5400 60  0000 C CNN
+	1    6700 5400
+	1    0    0    -1
+$EndComp
+$Comp
+L KFC-012-7.3 SW2
+U 1 1 5780DBBB
+P 7800 5400
+F 0 "SW2" H 7800 5050 60  0000 C CNN
+F 1 "KFC-012-7.3" H 7800 5750 60  0000 C CNN
+F 2 "tfhSwitches:KFC-012-7.3" H 7800 5400 60  0001 C CNN
+F 3 "" H 7800 5400 60  0000 C CNN
+	1    7800 5400
+	1    0    0    -1
+$EndComp
+$Comp
+L KFC-012-7.3 SW3
+U 1 1 5780DC01
+P 8900 5400
+F 0 "SW3" H 8900 5050 60  0000 C CNN
+F 1 "KFC-012-7.3" H 8900 5750 60  0000 C CNN
+F 2 "tfhSwitches:KFC-012-7.3" H 8900 5400 60  0001 C CNN
+F 3 "" H 8900 5400 60  0000 C CNN
+	1    8900 5400
+	1    0    0    -1
+$EndComp
+$Comp
+L KFC-012-7.3 SW4
+U 1 1 5780DC56
+P 10000 5400
+F 0 "SW4" H 10000 5050 60  0000 C CNN
+F 1 "KFC-012-7.3" H 10000 5750 60  0000 C CNN
+F 2 "tfhSwitches:KFC-012-7.3" H 10000 5400 60  0001 C CNN
+F 3 "" H 10000 5400 60  0000 C CNN
+	1    10000 5400
+	1    0    0    -1
+$EndComp
+Wire Wire Line
+	6250 5600 6250 5850
+Wire Wire Line
+	7150 5600 7150 5800
+Wire Wire Line
+	7150 5800 6250 5800
+Connection ~ 6250 5800
+Wire Wire Line
+	7350 5600 7350 5850
+Wire Wire Line
+	7350 5800 8250 5800
+Wire Wire Line
+	8250 5800 8250 5600
+Connection ~ 7350 5800
+Wire Wire Line
+	8450 5600 8450 5850
+Wire Wire Line
+	8450 5800 9350 5800
+Wire Wire Line
+	9350 5800 9350 5600
+Connection ~ 8450 5800
+Wire Wire Line
+	9550 5600 9550 5850
+Wire Wire Line
+	9550 5800 10450 5800
+Wire Wire Line
+	10450 5800 10450 5600
+Connection ~ 9550 5800
+NoConn ~ 7150 5200
+Wire Wire Line
+	9350 5200 9350 4650
+Wire Wire Line
+	10450 5200 10450 4650
+NoConn ~ 8450 5200
+NoConn ~ 9550 5200
+NoConn ~ 8250 5200
+NoConn ~ 8000 7700
 $EndSCHEMATC

Commit message: Updated missing libs
Parts:
- BT1: symbol Battery -> Battery-RESCUE-copyMe84
- D1, D2, D3, D4: symbol LED -> LED-RESCUE-copyMe84
Changed lines of the file:
@@
 EESchema Schematic File Version 2
+LIBS:copyMe84-rescue
 LIBS:power
 LIBS:device
@@
 $EndComp
 $Comp
-L LED D1
+L LED-RESCUE-copyMe84 D1
 U 1 1 5730C94B
 P 7000 3850
@@
 $EndComp
 $Comp
-L LED D2
+L LED-RESCUE-copyMe84 D2
 U 1 1 5730CD43
 P 7350 3850
@@
 $EndComp
 $Comp
-L LED D3
+L LED-RESCUE-copyMe84 D3
 U 1 1 5730CD7A
 P 7700 3850
@@
 $EndComp
 $Comp
-L LED D4
+L LED-RESCUE-copyMe84 D4
 U 1 1 5730CDAC
 P 8050 3850
@@
 SPEAKER
 $Comp
-L Battery BT1
+L Battery-RESCUE-copyMe84 BT1
 U 1 1 573111F5
 P 2150 3900

Commit message: V2.1
Changed lines of the file:
@@
 Wire Wire Line
 	5050 4350 6000 4350
-Wire Wire Line
-	5050 4550 6000 4550
-Wire Wire Line
-	5050 4450 6000 4450
 Text Label 5300 4250 0    60   ~ 0
 ledRED
@@
 	2550 4550 2550 4750
 Connection ~ 2550 4550
-NoConn ~ 5050 4050
 NoConn ~ 5050 3450
 NoConn ~ 5050 3350
@@
 Text Label 10450 5050 1    60   ~ 0
 swGREEN
+Text Label 5300 4050 0    60   ~ 0
+ledGREEN
 Text Label 5300 4450 0    60   ~ 0
-ledGREEN
-Text Label 5300 4550 0    60   ~ 0
 ledYELLOW
 Text Label 5300 3550 0    60   ~ 0
@@
 NoConn ~ 8250 5200
 NoConn ~ 8000 7700
+Wire Wire Line
+	5050 4050 6000 4050
+Wire Wire Line
+	5050 4450 6000 4450
+NoConn ~ 5050 4550
 $EndSCHEMATC
